File: hardware/soil-moisture-sensor.kicad_sch (KiCad schematic)
At the start: 22 parts

Commit message: schematic pretty much done
Parts:
- added D10, D9: (no value), symbol Device:LED
- added D2: (no value), symbol Diode:ESD9B3.3ST5G
- added D3, D5: ESD9B3.3ST5G, Diode_SMD:D_SOD-923, symbol Diode:ESD9B3.3ST5G
- added D4: (no value), symbol Device:D_Schottky
- added Q1: (no value), symbol Device:Q_NPN_BEC
- added Q2: Q_NPN_BEC, symbol Device:Q_NPN_BEC
- added R10, R11, R12, R3, R4, R6, R7: (no value), symbol Device:R
- added R8: 2k, symbol Device:R
- added U2: (no value), symbol Interface_USB:CP2102N-Axx-xQFN24
- gave numbers to parts that had none: 16
Connections:
- net SENSOR-IN is gone; now on net SENSOR_IN: R1.2
- net SENSOR-OUT is gone; now on net SENSOR_OUT: C2.1, D1.1 (K), D6.1 (K), R2.2
- net +3V3: now also D10.2 (A), D9.2 (A), R8.1, U2.5 (VIO), U2.6 (VDD)
- net EN: now also Q1.3 (C)
- net GND: now also C3.2, J1.5 (GND), J1.6 (Shield), U1.1 (GND), U3.1 (GND), U3.15 (GND), U3.38 (GND), U3.39 (GND), D2.1 (A1), D3.1 (A1), D5.1 (A1), R7.1, U2.2 (GND), U2.25 (GND)
- net IO0: now also Q2.3 (C)
- net USB_5V: now reaches J1.1 (VBUS)
- net USB_5V: now also D2.2 (A2), D4.2 (A), R6.1
- net USB_DM: now reaches J1.2 (D-)
- net USB_DM: now also D5.2 (A2), U2.4 (D-)
- net USB_DP: now reaches J1.3 (D+)
- net USB_DP: now also D3.2 (A2), U2.3 (D+)
- net SENSOR_OUT: now reaches U3.14 (IO12)
- net SENSOR_IN: now reaches U3.29 (IO5)
- net RXD: now reaches U3.34 (RXD0/IO3)
- net RXD: now also U2.20 (RXD)
- net TXD: now reaches U3.35 (TXD0/IO1)
- net TXD: now also U2.21 (TXD)
- new net: Q2.1 (B), R4.1
- new net: D9.1 (K), R11.2
- new net: R10.1, U2.15 (~{SUSPEND})
- new net: R8.2, U2.9 (~{RST})
- new net: R12.1, U2.13 (~{RXT}/GPIO.1)
- new net: R11.1, U2.14 (~{TXT}/GPIO.0)
- new net: R6.2, R7.2, U2.8 (VBUS)
- new net: D10.1 (K), R12.2
- new net: Q1.1 (B), R3.1
- new net DTR: Q2.2 (E), R3.2, U2.23 (~{DTR})
- new net RTS: Q1.2 (E), R4.2, U2.19 (~{RTS})
- new net VBUS: D4.1 (K)
Other:
- moved on the sheet: D8, R5
