File: hardware/_autosave-soil-moisture-sensor.kicad_sch (KiCad schematic)
At the start: 35 parts, among them J1 USB_B_Micro, Q1 Q_NPN_BEC, Q2 Q_NPN_BEC, SW1 SW_Push, SW2 SW_Push, U2 CP2102N-Axx-xQFN24, U3 ESP32-WROOM-32D

Commit message: placement pretty much done
Parts:
- R1: value 10K -> (none)
Changed lines of the file:
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@@
       (effects (font (size 1.27 1.27)) (justify left))
     )
-    (property "Value" "10K" (id 1) (at 39.37 167.64 90)
+    (property "Value" "" (id 1) (at 39.37 167.64 90)
       (effects (font (size 1.27 1.27)) (justify left))
     )
